File: Hardware/PCB/mark_1/M24C64_v1.sch (EAGLE design)
At the start: 2 parts, among them IC1 M24C64

Commit message: 
Parts:
- added JP1: (no value), mark_1:PINHD-1X4
Connections:
- net +5V: now also JP1.1
- net GND: now also JP1.4
- net SCL: now also JP1.2
- net SDA: now also JP1.3
Changed lines of the file:
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@@
 <part name="GND2" library="mark_1" deviceset="GND" device=""/>
 <part name="GND3" library="mark_1" deviceset="GND" device=""/>
+<part name="JP1" library="mark_1" deviceset="PINHD-1X4" device=""/>
+<part name="P+3" library="mark_1" deviceset="+5V" device=""/>
+<part name="GND4" library="mark_1" deviceset="GND" device=""/>
 </parts>
 <sheets>
@@
 <instance part="GND2" gate="1" x="-5.08" y="12.7"/>
 <instance part="GND3" gate="1" x="45.72" y="17.78"/>
+<instance part="JP1" gate="A" x="63.5" y="20.32"/>
+<instance part="P+3" gate="1" x="53.34" y="30.48" smashed="yes">
+<attribute name="VALUE" x="55.88" y="33.02" size="1.778" layer="96" rot="R180"/>
+</instance>
+<instance part="GND4" gate="1" x="53.34" y="12.7"/>
 </instances>
 <busses>
@@
 <wire x1="30.48" y1="25.4" x2="33.02" y2="25.4" width="0.1524" layer="91"/>
 <wire x1="33.02" y1="25.4" x2="33.02" y2="27.94" width="0.1524" layer="91"/>
+</segment>
+<segment>
+<pinref part="JP1" gate="A" pin="1"/>
+<pinref part="P+3" gate="1" pin="+5V"/>
+<wire x1="53.34" y1="27.94" x2="53.34" y2="25.4" width="0.1524" layer="91"/>
+<wire x1="53.34" y1="25.4" x2="60.96" y2="25.4" width="0.1524" layer="91"/>
 </segment>
 </net>
@@
 <wire x1="45.72" y1="22.86" x2="45.72" y2="20.32" width="0.1524" layer="91"/>
 </segment>
+<segment>
+<pinref part="JP1" gate="A" pin="4"/>
+<pinref part="GND4" gate="1" pin="GND"/>
+<wire x1="53.34" y1="15.24" x2="53.34" y2="17.78" width="0.1524" layer="91"/>
+<wire x1="53.34" y1="17.78" x2="60.96" y2="17.78" width="0.1524" layer="91"/>
+</segment>
 </net>
 <net name="SCL" class="0">
@@
 <wire x1="30.48" y1="20.32" x2="38.1" y2="20.32" width="0.1524" layer="91"/>
 <label x="33.02" y="20.32" size="1.778" layer="95"/>
+</segment>
+<segment>
+<pinref part="JP1" gate="A" pin="2"/>
+<wire x1="60.96" y1="22.86" x2="50.8" y2="22.86" width="0.1524" layer="91"/>
+<label x="50.8" y="22.86" size="1.778" layer="95"/>
 </segment>
 </net>
@@
 <label x="33.02" y="17.78" size="1.778" layer="95"/>
 </segment>
+<segment>
+<pinref part="JP1" gate="A" pin="3"/>
+<wire x1="60.96" y1="20.32" x2="50.8" y2="20.32" width="0.1524" layer="91"/>
+<label x="50.8" y="20.32" size="1.778" layer="95"/>
+</segment>
 </net>
