File: Hardware/PCB/mark_1/XBee_v1.sch (EAGLE design)
At the start: 12 parts, among them IC1 4050D, IC2 LM1117S

Commit message: 
Parts:
- removed C2, C3: 100uF, mark_1:CPOL-EUPD
- added JP2: TXD, mark_1:PINHD-1X1
- added JP3: RXD, mark_1:PINHD-1X1
- added JP4: RST, mark_1:PINHD-1X1
- added JP5: RSSI, mark_1:PINHD-1X1
- added JP6: DTR, mark_1:PINHD-1X1
- added JP7: CTS, mark_1:PINHD-1X1
- added JP8: RTS, mark_1:PINHD-1X1
- IC1: value 4050D -> 4050
- LED1, LED2: device mark_1:LED0805 -> mark_1:LED3MM
Connections:
- net +3V3: no longer C2.+
- net CTS: now also JP7.1
- net DTR: now also IC1A.I, JP6.1; no longer IC1C.I
- net GND: no longer C2.-, C3.-
- net N$1: no longer C3.+
- net N$3: now also IC1C.O; no longer IC1A.O
- net N$7: now also IC1A.O; no longer IC1C.O
- net RESET: now also JP4.1
- net RSSI: now also JP5.1
- net RTS: now also JP8.1
- net RXD: now also IC1C.I, JP3.1; no longer IC1A.I
- net TXD: now also JP2.1
Other:
- moved on the sheet: IC1A, IC1C
Changed lines of the file:
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@@
 </classes>
 <parts>
-<part name="IC1" library="mark_1" deviceset="4050" device="D"/>
+<part name="IC1" library="mark_1" deviceset="4050" device="D" value="4050"/>
 <part name="C1" library="mark_1" deviceset="C-EU" device="C0805K" value="100nF"/>
 <part name="IC2" library="mark_1" deviceset="LM1117" device="S"/>
-<part name="LED1" library="mark_1" deviceset="LED" device="0805"/>
+<part name="LED1" library="mark_1" deviceset="LED" device="3MM"/>
 <part name="R1" library="mark_1" deviceset="R-EU_" device="R0805"/>
 <part name="D1" library="mark_1" deviceset="S1M" device=""/>
@@
 <part name="GND2" library="mark_1" deviceset="GND" device=""/>
 <part name="+3V1" library="mark_1" deviceset="+3V3" device=""/>
-<part name="C2" library="mark_1" deviceset="CPOL-EU" device="PD" value="100uF"/>
 <part name="P+1" library="mark_1" deviceset="+5V" device=""/>
 <part name="JP1" library="mark_1" deviceset="PINHD-1X2" device=""/>
@@
 <part name="GND4" library="mark_1" deviceset="GND" device=""/>
 <part name="R2" library="mark_1" deviceset="R-EU_" device="R0805"/>
-<part name="LED2" library="mark_1" deviceset="LED" device="0805"/>
+<part name="LED2" library="mark_1" deviceset="LED" device="3MM"/>
 <part name="GND5" library="mark_1" deviceset="GND" device=""/>
 <part name="+3V3" library="mark_1" deviceset="+3V3" device=""/>
 <part name="GND6" library="mark_1" deviceset="GND" device=""/>
-<part name="C3" library="mark_1" deviceset="CPOL-EU" device="PD" value="100uF"/>
+<part name="JP2" library="mark_1" deviceset="PINHD-1X1" device="" value="TXD"/>
+<part name="JP3" library="mark_1" deviceset="PINHD-1X1" device="" value="RXD"/>
+<part name="JP4" library="mark_1" deviceset="PINHD-1X1" device="" value="RST"/>
+<part name="JP5" library="mark_1" deviceset="PINHD-1X1" device="" value="RSSI"/>
+<part name="JP6" library="mark_1" deviceset="PINHD-1X1" device="" value="DTR"/>
+<part name="JP7" library="mark_1" deviceset="PINHD-1X1" device="" value="CTS"/>
+<part name="JP8" library="mark_1" deviceset="PINHD-1X1" device="" value="RTS"/>
 </parts>
 <sheets>
@@
 </plain>
 <instances>
-<instance part="IC1" gate="A" x="22.86" y="53.34"/>
-<instance part="IC1" gate="B" x="22.86" y="40.64"/>
-<instance part="IC1" gate="C" x="22.86" y="17.78"/>
 <instance part="IC1" gate="D" x="22.86" y="2.54"/>
 <instance part="C1" gate="G$1" x="73.66" y="86.36" rot="R180"/>
@@
 <instance part="GND2" gate="1" x="30.48" y="76.2"/>
 <instance part="+3V1" gate="G$1" x="43.18" y="99.06"/>
-<instance part="C2" gate="G$1" x="43.18" y="88.9"/>
 <instance part="P+1" gate="1" x="10.16" y="99.06"/>
 <instance part="JP1" gate="G$1" x="5.08" y="88.9"/>
@@
 <instance part="+3V3" gate="G$1" x="66.04" y="96.52"/>
 <instance part="GND6" gate="1" x="66.04" y="76.2"/>
-<instance part="C3" gate="G$1" x="20.32" y="88.9"/>
+<instance part="JP2" gate="G$1" x="0" y="60.96" rot="R180"/>
+<instance part="JP3" gate="G$1" x="0" y="53.34" rot="R180"/>
+<instance part="JP4" gate="G$1" x="0" y="40.64" rot="R180"/>
+<instance part="JP5" gate="G$1" x="0" y="30.48" rot="R180"/>
+<instance part="JP6" gate="G$1" x="0" y="17.78" rot="R180"/>
+<instance part="JP7" gate="G$1" x="0" y="10.16" rot="R180"/>
+<instance part="JP8" gate="G$1" x="0" y="2.54" rot="R180"/>
+<instance part="IC1" gate="A" x="22.86" y="17.78"/>
+<instance part="IC1" gate="B" x="22.86" y="40.64"/>
+<instance part="IC1" gate="C" x="22.86" y="53.34"/>
 </instances>
 <busses>
@@
 <junction x="30.48" y="81.28"/>
 <wire x1="30.48" y1="81.28" x2="30.48" y2="78.74" width="0.1524" layer="91"/>
-<pinref part="C2" gate="G$1" pin="-"/>
-<wire x1="30.48" y1="81.28" x2="43.18" y2="81.28" width="0.1524" layer="91"/>
-<wire x1="43.18" y1="81.28" x2="43.18" y2="83.82" width="0.1524" layer="91"/>
 <pinref part="JP1" gate="G$1" pin="2"/>
 <wire x1="2.54" y1="88.9" x2="10.16" y2="88.9" width="0.1524" layer="91"/>
 <wire x1="10.16" y1="88.9" x2="10.16" y2="81.28" width="0.1524" layer="91"/>
-<wire x1="10.16" y1="81.28" x2="20.32" y2="81.28" width="0.1524" layer="91"/>
-<junction x="20.32" y="81.28"/>
-<wire x1="20.32" y1="81.28" x2="30.48" y2="81.28" width="0.1524" layer="91"/>
-<pinref part="C3" gate="G$1" pin="-"/>
-<wire x1="20.32" y1="83.82" x2="20.32" y2="81.28" width="0.1524" layer="91"/>
+<wire x1="10.16" y1="81.28" x2="30.48" y2="81.28" width="0.1524" layer="91"/>
 </segment>
 <segment>
@@
 <wire x1="38.1" y1="91.44" x2="43.18" y2="91.44" width="0.1524" layer="91"/>
 <wire x1="43.18" y1="91.44" x2="43.18" y2="96.52" width="0.1524" layer="91"/>
-<junction x="43.18" y="91.44"/>
-<pinref part="C2" gate="G$1" pin="+"/>
 </segment>
 <segment>
@@
 <net name="N$3" class="0">
 <segment>
-<pinref part="IC1" gate="A" pin="O"/>
 <pinref part="U$1" gate="G$1" pin="DIN"/>
 <wire x1="33.02" y1="53.34" x2="55.88" y2="53.34" width="0.1524" layer="91"/>
+<pinref part="IC1" gate="C" pin="O"/>
 </segment>
 </net>
 <net name="N$4" class="0">
 <segment>
-<pinref part="IC1" gate="B" pin="O"/>
 <wire x1="33.02" y1="40.64" x2="35.56" y2="40.64" width="0.1524" layer="91"/>
 <wire x1="35.56" y1="40.64" x2="35.56" y2="48.26" width="0.1524" layer="91"/>
 <pinref part="U$1" gate="G$1" pin="RESET"/>
 <wire x1="35.56" y1="48.26" x2="55.88" y2="48.26" width="0.1524" layer="91"/>
+<pinref part="IC1" gate="B" pin="O"/>
 </segment>
 </net>
@@
 <wire x1="38.1" y1="30.48" x2="2.54" y2="30.48" width="0.1524" layer="91"/>
 <label x="2.54" y="30.48" size="1.778" layer="95"/>
+<pinref part="JP5" gate="G$1" pin="1"/>
 </segment>
 </net>
@@
 <net name="N$7" class="0">
 <segment>
-<pinref part="IC1" gate="C" pin="O"/>
 <wire x1="33.02" y1="17.78" x2="48.26" y2="17.78" width="0.1524" layer="91"/>
 <wire x1="48.26" y1="17.78" x2="48.26" y2="38.1" width="0.1524" layer="91"/>
 <pinref part="U$1" gate="G$1" pin="DTR"/>
 <wire x1="48.26" y1="38.1" x2="55.88" y2="38.1" width="0.1524" layer="91"/>
+<pinref part="IC1" gate="A" pin="O"/>
 </segment>
 </net>
@@
 <net name="RXD" class="0">
 <segment>
-<pinref part="IC1" gate="A" pin="I"/>
 <wire x1="12.7" y1="53.34" x2="2.54" y2="53.34" width="0.1524" layer="91"/>
 <label x="2.54" y="53.34" size="1.778" layer="95"/>
+<pinref part="JP3" gate="G$1" pin="1"/>
+<pinref part="IC1" gate="C" pin="I"/>
 </segment>
 </net>
 <net name="RESET" class="0">
 <segment>
-<pinref part="IC1" gate="B" pin="I"/>
 <wire x1="12.7" y1="40.64" x2="2.54" y2="40.64" width="0.1524" layer="91"/>
 <label x="2.54" y="40.64" size="1.778" layer="95"/>
+<pinref part="JP4" gate="G$1" pin="1"/>
+<pinref part="IC1" gate="B" pin="I"/>
 </segment>
 </net>
 <net name="DTR" class="0">
 <segment>
-<pinref part="IC1" gate="C" pin="I"/>
 <wire x1="12.7" y1="17.78" x2="2.54" y2="17.78" width="0.1524" layer="91"/>
 <label x="2.54" y="17.78" size="1.778" layer="95"/>
+<pinref part="JP6" gate="G$1" pin="1"/>
+<pinref part="IC1" gate="A" pin="I"/>
 </segment>
 </net>
@@
 <wire x1="12.7" y1="2.54" x2="2.54" y2="2.54" width="0.1524" layer="91"/>
 <label x="2.54" y="2.54" size="1.778" layer="95"/>
+<pinref part="JP8" gate="G$1" pin="1"/>
 </segment>
 </net>
@@
 <wire x1="35.56" y1="60.96" x2="2.54" y2="60.96" width="0.1524" layer="91"/>
 <label x="2.54" y="60.96" size="1.778" layer="95"/>
+<pinref part="JP2" gate="G$1" pin="1"/>
 </segment>
 </net>
@@
 <wire x1="99.06" y1="10.16" x2="2.54" y2="10.16" width="0.1524" layer="91"/>
 <label x="2.54" y="10.16" size="1.778" layer="95"/>
+<pinref part="JP7" gate="G$1" pin="1"/>
 </segment>
 </net>
 <net name="N$1" class="0">
 <segment>
-<pinref part="C3" gate="G$1" pin="+"/>
-<junction x="20.32" y="91.44"/>
 <pinref part="D1" gate="D1" pin="C"/>
-<wire x1="17.78" y1="91.44" x2="20.32" y2="91.44" width="0.1524" layer="91"/>
 <pinref part="IC2" gate="G$1" pin="IN"/>
-<wire x1="22.86" y1="91.44" x2="20.32" y2="91.44" width="0.1524" layer="91"/>
-</segment>
-</net>
+<wire x1="22.86" y1="91.44" x2="17.78" y2="91.44" width="0.1524" layer="91"/>
+</segment>
+</net>
