File: Hardware/PCB/mark_2/demeter_v27.brd (EAGLE design)
At the start: 90 x 56 mm, 70 parts, among them IC1 4050, IC2 LM1117-5.0, IC3 LM1117-3.3, IC5 MCP3424, IC6 MCP23017SO, IC8 ATMEGA32U4-AU, Q1 IRLML6402, Q3 IRLML6402, Q5 IRLML6402

Commit message: 
Parts:
- removed C4: 22uF, mark_2:PANASONIC_D
- moved R3 23.9 mm to (41.3, 20.3), flipped to the bottom
- moved JP1 21.6 mm to (46.2, 20.3)
- moved C8 14.5 mm to (52.1, 40.6), turned to 45 degrees
- moved C1 10.5 mm to (52.6, 27.1), turned to 135 degrees
- moved C5 7.73 mm to (30.5, 36.8)
- moved D1 7.34 mm to (11.3, 40.6), turned to 270 degrees
- moved C11 6.60 mm to (20.3, 26.3), turned to 180 degrees
- moved C10 6.48 mm to (32.4, 27.9)
- moved C9 6.48 mm to (32.4, 33.0)
- moved IC3 6.48 mm to (27.9, 48.3)
- moved IC8 5.08 mm to (46.4, 34.4), turned to 45 degrees
- moved IC1 4.58 mm to (20.3, 17.1)
- moved U$1 2.54 mm to (22.9, 26.7)
- moved Q9 2.54 mm to (27.9, 30.5)
- moved IC2 1.80 mm to (17.8, 48.3)
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Connections:
- net +12V: no longer C4.+
- net GND: no longer C4.-
Routing:
- net N$27: track 59.9 -> 18.4 mm, vias 4 -> 0
- net +3V3: track 261.6 -> 221.8 mm, vias 9 -> 8
- net RSSI: track 36.6 -> 0.00 mm, vias 3 -> 0
- net SCL: track 37.5 -> 62.8 mm
- net D-: track 13.4 -> 35.5 mm, vias 1 -> 3
- net MOSI: track 29.5 -> 8.07 mm, vias 1 -> 0
- net SCK: track 32.3 -> 11.8 mm, vias 1 -> 0
- net RST: track 3.05 -> 22.5 mm
- net GND: track 471.4 -> 490.7 mm, vias 8 -> 9
- net RTS: track 84.8 -> 68.2 mm
- net +5V: track 281.3 -> 296.7 mm, vias 8 -> 6
- net MISO: track 22.1 -> 10.1 mm, vias 2 -> 0
- net +12V: track 49.1 -> 37.8 mm, vias 4 -> 2
- net VBUS: track 27.6 -> 38.2 mm
- net D+: track 11.4 -> 21.8 mm
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