File: Hardware/PCB/mark_2/demeter_v27.sch (EAGLE design)
At the start: 69 parts, among them IC1 4050, IC2 LM1117-5.0, IC3 LM1117-3.3, IC5 MCP3424, IC6 MCP23017SO, IC8 ATMEGA32U4-AU, Q1 IRLML6402, Q2 IRLML6402, Q3 IRLML6402, Q4 IRLML6402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

Commit message: 
Parts:
- removed C4: 22uF, mark_2:CPOL-EUPD
Connections:
- net +12V: no longer C4.+
- net GND: no longer C4.-
Changed lines of the file:
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@@
 <part name="D1" library="mark_2" deviceset="S1M" device=""/>
 <part name="C3" library="mark_2" deviceset="CPOL-EU" device="PD" value="100uF"/>
-<part name="C4" library="mark_2" deviceset="CPOL-EU" device="PD" value="22uF"/>
 <part name="IC3" library="mark_2" deviceset="LM1117" device="DT" value="LM1117-3.3"/>
 <part name="C5" library="mark_2" deviceset="CPOL-EU" device="PD" value="100uF"/>
@@
 <instance part="D1" gate="D1" x="276.86" y="48.26"/>
 <instance part="C3" gate="G$1" x="320.04" y="43.18"/>
-<instance part="C4" gate="G$1" x="294.64" y="12.7"/>
 <instance part="IC3" gate="G$1" x="307.34" y="17.78" smashed="yes">
 <attribute name="NAME" x="302.26" y="22.86" size="1.778" layer="95"/>
@@
 </segment>
 <segment>
-<pinref part="C4" gate="G$1" pin="-"/>
-<wire x1="294.64" y1="7.62" x2="294.64" y2="5.08" width="0.1524" layer="91"/>
 <pinref part="C5" gate="G$1" pin="-"/>
-<wire x1="294.64" y1="5.08" x2="307.34" y2="5.08" width="0.1524" layer="91"/>
 <wire x1="307.34" y1="5.08" x2="320.04" y2="5.08" width="0.1524" layer="91"/>
 <wire x1="320.04" y1="5.08" x2="320.04" y2="7.62" width="0.1524" layer="91"/>
@@
 <pinref part="IC3" gate="G$1" pin="IN"/>
 <wire x1="299.72" y1="17.78" x2="294.64" y2="17.78" width="0.1524" layer="91"/>
-<pinref part="C4" gate="G$1" pin="+"/>
-<wire x1="294.64" y1="17.78" x2="294.64" y2="15.24" width="0.1524" layer="91"/>
-<junction x="294.64" y="17.78"/>
 <pinref part="P+4" gate="1" pin="+12V"/>
 <wire x1="294.64" y1="20.32" x2="294.64" y2="17.78" width="0.1524" layer="91"/>
