File: Hardware/PCB/mark_2/demeter_v28-TSSOP.sch (EAGLE design)
At the start: 68 parts, among them IC1 MCP3424, IC2 MCP23017, IC3 LM1117-5.0, IC4 LM1117-3.3, IC5 4050, IC6 XBEE, IC7 ATMEGA32U4, Q1 IRLML6402, Q2 IRLML6402, Q3 IRLML6402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

Commit message: 
Other:
- note added: "ADC & I/O EXPANDER"
- note added: "MICROCONTROLLER"
- note added: "POWER"
- note added: "ZIGBEE"
- moved on the sheet: C1, C10, C2, C3, C4, C5, C6, C7, C8, C9, CN1, D1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
